Commit message: Update robot.urdf

File: robot_description/urdf/robot.urdf (robot description, URDF)
Before this commit: robot robot_arm, 3 links, 2 joints
Links:
- link link2: geometry collision mesh filename=package://robot_description/meshes/Part6.6.STL scale=0.001 0.001 0.001; visual mesh filename=package://robot_description/meshes/Part6.6.STL scale=0.001 0.001 0.001
Joints:
- joint joint2: limit lower=0 upper=0.02 effort=100 velocity=1 -> lower=0 upper=0.022 effort=100 velocity=1
